File: TinkerLink.kicad_sch (KiCad schematic)
At the start: 31 parts, among them J1 Conn_01x06_Pin, Q2 MMBT2222A, Q3 SQS411ENW-T1_GE3, Q4 SQS411ENW-T1_GE3, SW1 TS-061D-250D4-P, U1 ESP-01F-2M, U16 INA228, U2 ME6211C33M5, U3 AP63203WU, U5 TPD2EUSB30A

Commit message: can't... stop... tweakin'...
Parts:
- removed C1, C2: 10uf, Capacitor_SMD:C_0603_1608Metric, symbol Device:C
- removed D1: ~, LCSCfootprints:LED-SMD_6P-L3.5-W3.5_SK6812MINIRGBW-WS-P6-A, symbol AC_LED:SK6812_mini_RGBW
- removed L1: W3000, LCSCfootprints:ANT-SMD_L7.0-W1.6, symbol ANT-SMD_L7.0-W1.6:W3000
- removed U2: ME6211C33M5, Package_TO_SOT_SMD:SOT-23-5, symbol Regulator_Linear:ME6211C33M5
Connections:
- net VbusX is gone; now on net Vbus: C5.1, Q3.1 (S), Q3.2 (S), Q3.3 (S), R1.1, R47.1, U16.9 (Vin-), U3.2 (EN), U3.3 (IN)
- no-connect marks 2 -> 3
Other:
- note added: "3v3 Vdd source"
- note added: "Vbus monitoring"
- note added: "Vbus switching"
- note added: "tinker:USB-A-USB-C"
- note removed: "LCSCfootprints:USB-A-SMD_USB-212-BCW"
- note removed: "Minimal 3v3 source"
- note removed: "Possible replacement 3v3 source"
- moved on the sheet: C3, C5, C6, C7, C8, C86, J1, L2, LED1, LOGO1, Q2, Q3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
