File: Hardware/TinkerLink.kicad_pcb (KiCad board)
At the start: 2 copper layers, 40 x 24 mm, 31 parts, among them J1 Conn_01x06_Pin, Q1 DMN32D2LDF, Q2 MMBT2222A, Q3 SQS411ENW-T1_GE3, Q4 SQS411ENW-T1_GE3, SW1 TS-061D-250D4-P, U1 ESP-01F-2M, U2 INA228, U3 AP63203WU, U4 TPD2EUSB30A

Commit message: Starting to prep for publication
Changed lines of the file:
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@@
 	(title_block
 		(title "TinkerLink")
-		(rev "0.0.6")
+		(rev "0.0.8")
 		(company "S. A. Miller")
 		(comment 1 "With much input by Austin's Creations")
